File: color_sensor_electrical/color_sensor_electrical.kicad_pcb (KiCad board)
At the start: 2 copper layers, 48 x 36 mm, 18 parts, among them J1 OLED_header, J2 FTDI_header, SW1 SW_SPDT, U1 ATmega328P-AU, U2 S-1133B50-U5T1U, U3 TCS3200D-TR, Y1 Resonator

Commit message: Almost ready to order board.
Parts:
- J1: footprint Connector_PinSocket_1.00mm:PinSocket_1x04_P1.00mm_Vertical -> Connector_PinSocket_2.54mm:PinSocket_1x04_P2.54mm_Vertical
- J2: footprint Connector_PinSocket_1.00mm:PinSocket_1x06_P1.00mm_Vertical -> Connector_PinSocket_2.54mm:PinSocket_1x06_P2.54mm_Vertical
- moved J2 5.52 mm to (145.5, 75.5)
- moved C5 1.41 mm to (145.7, 79.0)
Routing:
- net Net-(BT3-Pad1): track 77.6 -> 22.7 mm
- net +5V: track 49.8 -> 36.6 mm
- net GND: track 34.8 -> 28.7 mm
- net PIN_A5: track 17.1 -> 18.3 mm
- net PIN_1_(TX): track 20.8 -> 20.0 mm
Other:
- board text added: "github.com/color-sensor v1.0 Elaine Jeffery"

Commit message: Added 3D models to PCB.
Parts:
- U2: footprint Package_TO_SOT_SMD:SOT-89-5_Handsoldering -> color_sensor_electrical:SOT-89-5_Handsoldering
Other:
- board text added: "github.com/duwaar/Pocket-Color-Sensor v1.0 Elaine Jeffery"
- board text removed: "github.com/color-sensor v1.0 Elaine Jeffery"
Changed lines of the file:
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@@
     (add_net RST)
+  )
+  (module color_sensor_electrical:SOT-89-5_Handsoldering (layer F.Cu)
+    (at 163.8 94.8 90)
+    (descr "SOT-89-5, http://www.e-devices.ricoh.co.jp/en/products/product_power/pkg/sot-89-5.pdf")
+    (tags SOT-89-5)
+    (attr smd)
+    (fp_text reference U2 (at 0 -3.5 90) (layer F.SilkS)
+      (effects (font (size 1 1) (thickness 0.15)))
+    )
+    (fp_text value S-1133B50-U5T1U (at 0 3.5 90) (layer F.Fab)
+      (effects (font (size 1 1) (thickness 0.15)))
+    )
+    (fp_text user %R (at 0.5 0) (layer F.Fab)
+      (effects (font (size 1 1) (thickness 0.15)))
+    )
+    (fp_line (start -3.85 2.5) (end -3.85 -2.5) (layer F.CrtYd) (width 0.05))
+    (fp_line (start -3.85 2.5) (end 3.85 2.5) (layer F.CrtYd) (width 0.05))
+    (fp_line (start 3.85 -2.5) (end -3.85 -2.5) (layer F.CrtYd) (width 0.05))
+    (fp_line (start 3.85 -2.5) (end 3.85 2.5) (layer F.CrtYd) (width 0.05))
+    (fp_line (start -0.25 -2.25) (end 1.25 -2.25) (layer F.Fab) (width 0.1))
+    (fp_line (start -1.25 2.25) (end -1.25 -1.25) (layer F.Fab) (width 0.1))
+    (fp_line (start 1.25 2.25) (end -1.25 2.25) (layer F.Fab) (width 0.1))
+    (fp_line (start 1.25 -2.25) (end 1.25 2.25) (layer F.Fab) (width 0.1))
+    (fp_line (start -1.25 -1.25) (end -0.25 -2.25) (layer F.Fab) (width 0.1))
+    (fp_line (start -1.36 2.36) (end -1.36 2.03) (layer F.SilkS) (width 0.12))
+    (fp_line (start -1.36 -2.36) (end -1.36 -2.03) (layer F.SilkS) (width 0.12))
+    (fp_line (start -1.36 -2.36) (end 1.36 -2.36) (layer F.SilkS) (width 0.12))
+    (fp_line (start 1.36 -2.36) (end 1.36 -2.03) (layer F.SilkS) (width 0.12))
+    (fp_line (start -3.54 -2.03) (end -1.36 -2.03) (layer F.SilkS) (width 0.12))
+    (fp_line (start 1.36 2.36) (end -1.36 2.36) (layer F.SilkS) (width 0.12))
+    (fp_line (start 1.36 2.03) (end 1.36 2.36) (layer F.SilkS) (width 0.12))
+    (pad 2 smd custom (at 0 0 90) (size 0.8 2) (layers F.Cu F.Paste F.Mask)
+      (net 2 GND) (zone_connect 2)
+      (options (clearance outline) (anchor rect))
+      (primitives
+        (gr_poly (pts
+           (xy -3.6 -0.5) (xy -0.9 -0.5) (xy -0.4 -1) (xy 0.4 -1) (xy 0.9 -0.5)
+           (xy 3.6 -0.5) (xy 3.6 0.5) (xy 0.9 0.5) (xy 0.4 1) (xy -0.4 1)
+           (xy -0.9 0.5) (xy -3.6 0.5)) (width 0))
+      ))
+    (pad 3 smd rect (at -2.35 1.5 90) (size 2.5 0.7) (layers F.Cu F.Paste F.Mask)
+      (net 2 GND))
+    (pad 1 smd rect (at -2.35 -1.5 90) (size 2.5 0.7) (layers F.Cu F.Paste F.Mask))
+    (pad 4 smd rect (at 2.35 1.5 90) (size 2.5 0.7) (layers F.Cu F.Paste F.Mask)
+      (net 4 "Net-(C2-Pad1)"))
+    (pad 5 smd rect (at 2.35 -1.5 90) (size 2.5 0.7) (layers F.Cu F.Paste F.Mask)
+      (net 5 +5V))
+    (model :color_sensor_3d_models:S1133_E.step
+      (at (xyz 0 0 0))
+      (scale (xyz 1 1 1))
+      (rotate (xyz 0 0 90))
+    )
   )
   (module Connector_PinSocket_2.54mm:PinSocket_1x04_P2.54mm_Vertical (layer F.Cu)
@@
       (net 33 PIN_4))
     (model ${KISYS3DMOD}/Package_SO.3dshapes/SOIC-8_3.9x4.9mm_P1.27mm.wrl
-      (at (xyz 0 0 0))
-      (scale (xyz 1 1 1))
-      (rotate (xyz 0 0 0))
-    )
-  )
-  (module Package_TO_SOT_SMD:SOT-89-5_Handsoldering (layer F.Cu)
-    (at 163.8 94.8 90)
-    (descr "SOT-89-5, http://www.e-devices.ricoh.co.jp/en/products/product_power/pkg/sot-89-5.pdf")
-    (tags SOT-89-5)
-    (attr smd)
-    (fp_text reference U2 (at 4.7 0 180) (layer F.SilkS)
-      (effects (font (size 1 1) (thickness 0.15)))
-    )
-    (fp_text value S-1133B50-U5T1U (at 0 3.5 90) (layer F.Fab)
-      (effects (font (size 1 1) (thickness 0.15)))
-    )
-    (fp_line (start -3.85 2.5) (end -3.85 -2.5) (layer F.CrtYd) (width 0.05))
-    (fp_line (start -3.85 2.5) (end 3.85 2.5) (layer F.CrtYd) (width 0.05))
-    (fp_line (start 3.85 -2.5) (end -3.85 -2.5) (layer F.CrtYd) (width 0.05))
-    (fp_line (start 3.85 -2.5) (end 3.85 2.5) (layer F.CrtYd) (width 0.05))
-    (fp_line (start -0.25 -2.25) (end 1.25 -2.25) (layer F.Fab) (width 0.1))
-    (fp_line (start -1.25 2.25) (end -1.25 -1.25) (layer F.Fab) (width 0.1))
-    (fp_line (start 1.25 2.25) (end -1.25 2.25) (layer F.Fab) (width 0.1))
-    (fp_line (start 1.25 -2.25) (end 1.25 2.25) (layer F.Fab) (width 0.1))
-    (fp_line (start -1.25 -1.25) (end -0.25 -2.25) (layer F.Fab) (width 0.1))
-    (fp_line (start -1.36 2.36) (end -1.36 2.03) (layer F.SilkS) (width 0.12))
-    (fp_line (start -1.36 -2.36) (end -1.36 -2.03) (layer F.SilkS) (width 0.12))
-    (fp_line (start -1.36 -2.36) (end 1.36 -2.36) (layer F.SilkS) (width 0.12))
-    (fp_line (start 1.36 -2.36) (end 1.36 -2.03) (layer F.SilkS) (width 0.12))
-    (fp_line (start -3.54 -2.03) (end -1.36 -2.03) (layer F.SilkS) (width 0.12))
-    (fp_line (start 1.36 2.36) (end -1.36 2.36) (layer F.SilkS) (width 0.12))
-    (fp_line (start 1.36 2.03) (end 1.36 2.36) (layer F.SilkS) (width 0.12))
-    (fp_text user %R (at 0.5 0) (layer F.Fab)
-      (effects (font (size 1 1) (thickness 0.15)))
-    )
-    (pad 2 smd custom (at 0 0 90) (size 0.8 2) (layers F.Cu F.Paste F.Mask)
-      (net 2 GND) (zone_connect 2)
-      (options (clearance outline) (anchor rect))
-      (primitives
-        (gr_poly (pts
-           (xy -3.6 -0.5) (xy -0.9 -0.5) (xy -0.4 -1) (xy 0.4 -1) (xy 0.9 -0.5)
-           (xy 3.6 -0.5) (xy 3.6 0.5) (xy 0.9 0.5) (xy 0.4 1) (xy -0.4 1)
-           (xy -0.9 0.5) (xy -3.6 0.5)) (width 0))
-      ))
-    (pad 3 smd rect (at -2.35 1.5 90) (size 2.5 0.7) (layers F.Cu F.Paste F.Mask)
-      (net 2 GND))
-    (pad 1 smd rect (at -2.35 -1.5 90) (size 2.5 0.7) (layers F.Cu F.Paste F.Mask))
-    (pad 4 smd rect (at 2.35 1.5 90) (size 2.5 0.7) (layers F.Cu F.Paste F.Mask)
-      (net 4 "Net-(C2-Pad1)"))
-    (pad 5 smd rect (at 2.35 -1.5 90) (size 2.5 0.7) (layers F.Cu F.Paste F.Mask)
-      (net 5 +5V))
-    (model ${KISYS3DMOD}/Package_TO_SOT_SMD.3dshapes/SOT-89-5.wrl
       (at (xyz 0 0 0))
       (scale (xyz 1 1 1))
@@
     )
   )
-  (gr_text "github.com/color-sensor\nv1.0\nElaine Jeffery" (at 134.1 105.3) (layer F.SilkS)
+  (gr_text "github.com/duwaar/Pocket-Color-Sensor\nv1.0\nElaine Jeffery" (at 134.1 105.3) (layer F.SilkS)
     (effects (font (size 1 1) (thickness 0.15)) (justify left))
   )
