File: color_sensor_electrical/color_sensor_electrical.sch (KiCad schematic (older format))
At the start: 20 parts, among them J1 OLED_header, J2 FTDI_header, SW1 SW_SPDT, U1 ATmega328P-AU, U2 S-1133B50-U5T1U, U3 TCS3200D-TR, Y1 Resonator

Commit message: Almost ready to order board.
Parts:
- J1: footprint Connector_PinSocket_1.00mm:PinSocket_1x04_P1.00mm_Vertical -> Connector_PinSocket_2.54mm:PinSocket_1x04_P2.54mm_Vertical
- J2: footprint Connector_PinSocket_1.00mm:PinSocket_1x06_P1.00mm_Vertical -> Connector_PinSocket_2.54mm:PinSocket_1x06_P2.54mm_Vertical
Changed lines of the file:
@@
 F 0 "J2" H 8350 3950 50  0000 L CNN
 F 1 "FTDI_header" H 7950 3850 50  0000 L CNN
-F 2 "Connector_PinSocket_1.00mm:PinSocket_1x06_P1.00mm_Vertical" H 8500 3500 50  0001 C CNN
+F 2 "Connector_PinSocket_2.54mm:PinSocket_1x06_P2.54mm_Vertical" H 8500 3500 50  0001 C CNN
 F 3 "~" H 8500 3500 50  0001 C CNN
 F 4 "bulk" H 8500 3500 50  0001 C CNN "Packaging"
@@
 F 0 "J1" H 8350 2700 50  0000 L CNN
 F 1 "OLED_header" H 8050 2600 50  0000 L CNN
-F 2 "Connector_PinSocket_1.00mm:PinSocket_1x04_P1.00mm_Vertical" H 8500 2400 50  0001 C CNN
+F 2 "Connector_PinSocket_2.54mm:PinSocket_1x04_P2.54mm_Vertical" H 8500 2400 50  0001 C CNN
 F 3 "~" H 8500 2400 50  0001 C CNN
 F 4 "~" H 8500 2400 50  0001 C CNN "Packaging"

Commit message: Added 3D models to PCB.
Parts:
- J1: footprint Connector_PinSocket_2.54mm:PinSocket_1x04_P2.54mm_Vertical -> color_sensor_electrical:PinSocket_1x04_P2.54mm_Vertical
- U2: footprint Package_TO_SOT_SMD:SOT-89-5_Handsoldering -> color_sensor_electrical:SOT-89-5_Handsoldering
Changed lines of the file:
@@
 F 0 "U2" H 7100 5365 50  0000 C CNN
 F 1 "S-1133B50-U5T1U" H 7100 5274 50  0000 C CNN
-F 2 "Package_TO_SOT_SMD:SOT-89-5_Handsoldering" H 7100 4950 50  0001 C CNN
+F 2 "color_sensor_electrical:SOT-89-5_Handsoldering" H 7100 4950 50  0001 C CNN
 F 3 "~" H 7100 4950 50  0001 C CNN
 F 4 "1662-2896-1-ND" H 7100 4950 50  0001 C CNN "S1PN"
@@
 F 0 "J1" H 8350 2700 50  0000 L CNN
 F 1 "OLED_header" H 8050 2600 50  0000 L CNN
-F 2 "Connector_PinSocket_2.54mm:PinSocket_1x04_P2.54mm_Vertical" H 8500 2400 50  0001 C CNN
+F 2 "color_sensor_electrical:PinSocket_1x04_P2.54mm_Vertical" H 8500 2400 50  0001 C CNN
 F 3 "~" H 8500 2400 50  0001 C CNN
 F 4 "~" H 8500 2400 50  0001 C CNN "Packaging"
